File: vidc_interposer1.sch (EAGLE design)
At the start: 28 parts, among them IC1 SN74ALVC164245, IC2 SN74ALVC164245, IC3 SN74ALVC164245, IC5 MCP1703CB

Commit message: Update schematics with licence
Other:
- note added: "CC BY-SA 3.0"
