File: vidc_interposer2-PTH.sch (EAGLE design)
At the start: 25 parts, among them IC1 SN74ALVC164245, IC2 SN74ALVC164245, IC3 SN74ALVC164245, U1 MIC5219 3.3V

Commit message: Update schematics with licence
Other:
- note added: "CC BY-SA 3.0"
Changed lines of the file:
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@@
 <text x="50.8" y="406.4" size="1.778" layer="91">PTH for A3000, slightly taller &amp; no upper socket!</text>
 <text x="495.3" y="33.02" size="1.778" layer="91">(For A3000/soldered VIDC)</text>
+<text x="487.68" y="27.94" size="1.778" layer="91">CC BY-SA 3.0</text>
 </plain>
 <instances>
